File: pcb/SolarKey.kicad_pcb (KiCad board)
At the start: 2 copper layers, 260.4 x 81 mm, 144 parts, among them SW1 RotaryEncoder_Switch, SW2 RotaryEncoder_Switch, U2 RP2040_Pro_Micro

Commit message: update kicad files
Connections:
- U2 pad 29: unconnected-(U2-GND-Pad29) -> Net-(U2-GND-Pad29)
- U2 pad 30: unconnected-(U2-5v-Pad30) -> +5V
- U2 pad 4: unconnected-(U2-GND-Pad4) -> Net-(U2-GND-Pad4)
- U2 pad 5: unconnected-(U2-GND-Pad5) -> Net-(U2-GND-Pad5)
Routing:
- net +5V: track 988.9 -> 1021.8 mm, vias 20 -> 22
- net Net-(D88-DOUT): track 38.8 -> 41.3 mm
