File: pcb/SolarKey.kicad_sch (KiCad schematic)
At the start: 144 parts, among them SW1 RotaryEncoder_Switch, SW2 RotaryEncoder_Switch, U2 RP2040_Pro_Micro

Commit message: update kicad files
Connections:
- net +5V: now also U2.30 (5v)
