File: PCB/Wind47v2.kicad_pcb (KiCad board)
At the start: 2 copper layers, 260.4 x 81 mm, 144 parts, among them SW1 RotaryEncoder_Switch, SW2 RotaryEncoder_Switch, U2 RP2040_Pro_Micro

Commit message: Update PCB net assignments and production files
Renamed and reordered several net assignments in Wind47v2.kicad_pcb to remove unused nets and improve clarity. Updated production STL and ZIP files, removed outdated backups, and added new 3D and PCB files. Journal updated with design changes for USB-C port and floor thickness adjustment.
Connections:
- U2 pad 29: Net-(U2-GND-Pad29) -> GND
- U2 pad 4: Net-(U2-GND-Pad4) -> GND
- U2 pad 5: Net-(U2-GND-Pad5) -> GND
Routing:
- net row0: track 322.3 -> 321.4 mm
- net row3: track 336.4 -> 335.4 mm
- net row2: track 334.3 -> 333.4 mm
- net row1: track 314.4 -> 313.5 mm
- added copper zone on B.Cu, net GND
- added copper zone on F.Cu, net GND
